File: boards/ATSAMR21-Breakout.brd (EAGLE design)
At the start: 27.6 x 50.8 mm, 26 parts, among them IC3 NCP4589DSN33T1G, IC4 ATSAMR21G18-MR210UA

Commit message: Added LED and re-routed chg-mgmt signals.
Parts:
- added LED1: (no value), led:CHIPLED_1206
- added R7: 220, SparkFun-Resistors:0805
- added SJ5, SJ6: SOLDERJUMPERTRACE, SparkFun-Retired:SJ_2S-TRACE
- added TP4, TP5, TP6: TPTP15R, testpad:TP15R
- TP1, TP2, TP3: value TPB2,54 -> TPTP15R; device testpad:B2,54 -> testpad:TP15R
Connections:
- new net N$6: LED1.A, SJ6.1
- new net N$7: R7.1, SJ6.2
- net 3.3V: now also SJ5.1, SJ5.2, TP4.TP, TP5.TP
- net ANT_DIV_P: now also TP6.TP; no longer SV2.3
- net CHG_STATUS: now also SV2.2; no longer SV2.1
- net GND: now also LED1.C, SV2.1
- net GPIO: now also R7.2
- net PWR_STAT: now also SV2.3; no longer SV2.2
Routing:
- net ANT_DIV_P: track 31.1 -> 3.56 mm, vias 0 -> 1
- net N$7: track 0.00 -> 21.5 mm
- net GND: track 180.8 -> 185.0 mm
- net N$6: track 0.00 -> 2.55 mm
- net GPIO: track 31.2 -> 33.6 mm, vias 1 -> 2
- net PWR_STAT: track 16.9 -> 14.7 mm
- net CHG_STATUS: track 17.9 -> 16.3 mm
- net 3.3V: track 67.4 -> 68.1 mm
- net RXD1: track 31.9 -> 31.3 mm
Other:
- board text added: "ATSAMR21 BREAKOUT V0.3"
- board text removed: "ANT_DIV"
- board text removed: "ATSAMR21 BREAKOUT V0.2"
