File: boards/ATSAMR21-Breakout.sch (EAGLE design)
At the start: 26 parts, among them IC3 NCP4589DSN33T1G, IC4 ATSAMR21G18-MR210UA

Commit message: Added LED and re-routed chg-mgmt signals.
Parts:
- added LED1: (no value), led:LEDCHIPLED_1206
- added R7: 220, SparkFun-Resistors:RESISTOR0805-RES
- added SJ5, SJ6: SOLDERJUMPERTRACE, SparkFun-Retired:SOLDERJUMPERTRACE
- added TP4, TP5, TP6: TPTP15R, testpad:TPTP15R
- TP1, TP2, TP3: value TPB2,54 -> TPTP15R; device testpad:TPB2,54 -> testpad:TPTP15R
Connections:
- new net N$6: LED1.A, SJ6.1
- new net N$7: R7.1, SJ6.2
- net 3.3V: now also SJ5.1, SJ5.2, TP4.TP, TP5.TP
- net ANT_DIV_P: now also TP6.TP; no longer SV2.3
- net CHG_STATUS: now also SV2.2; no longer SV2.1
- net GND: now also LED1.C, SV2.1
- net GPIO: now also R7.2
- net PWR_STAT: now also SV2.3; no longer SV2.2
Other:
- moved on the sheet: SJ1, SJ2, TP1, TP2, TP3
